Commit message: Update cyton_gamma_1500.urdf
Added collisions meshes

File: cyton_gamma_1500_description/cyton_gamma_1500.urdf (robot description, URDF)
Before this commit: robot cyton_gamma_1500, 10 links, 9 joints
Links:
- link elbow_pitch: geometry collision sphere radius=0.055; visual mesh filename=package://cyton_gamma_1500_description/meshes/elbow_pitch.d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
- link elbow_yaw: geometry collision sphere radius=0.05; visual mesh filename=package://cyton_gamma_1500_description/meshes/elbow_yaw.dae
- link shoulder_pitch: geometry collision sphere radius=0.055; visual mesh filename=package://cyton_gamma_1500_description/meshes/shoulder_pitc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
- link shoulder_roll: geometry collision box size=0.09829 0.046 0.08392; visual mesh filename=package://cyton_gamma_1500_description/meshes/shoulder_roll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
- link shoulder_yaw: geometry collision sphere radius=0.055; visual mesh filename=package://cyton_gamma_1500_description/meshes/shoulder_yaw.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
- link wrist_pitch: geometry collision box size=0.07 0.06 0.11; visual mesh filename=package://cyton_gamma_1500_description/meshes/wrist_pitch.d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
- link wrist_roll: geometry collision box size=0.08 0.06 0.08; visual mesh filename=package://cyton_gamma_1500_description/meshes/wrist_roll.dae
